File: hw/main/main.kicad_pcb (KiCad board)
At the start: 2 copper layers, 91.3 x 100 mm, 42 parts, among them J1 Control A, J2 Control Pwr, J3 LCD, J4 Power, J5 Control D, J6 DAC Out, U1 MCP4821, U2 MCP3208, U3 LM4040C30, U4 LM4040C30, U5 TL072, U6 LMR50410

Commit message: kinda finsihed main
Parts:
- added LOGO1: Crankery, lama:crankery_small, F.Cu at (35.5, 120.4)
- added LOGO2: Monk, lama:monk, B.Cu at (71.1, 73.2)
- moved J1 2.54 mm to (88.9, 52.2)
- moved J5 2.54 mm to (88.9, 36.9)
- moved J6 2.54 mm to (88.9, 29.6)
- moved C9 0.51 mm to (52.6, 52.1)
Routing:
- net +5V: track 0.00 -> 207.8 mm, vias 0 -> 7
- net +3.3V: track 0.00 -> 156.0 mm, vias 0 -> 6
- net /LCD_SCL: track 0.00 -> 141.3 mm, vias 0 -> 3
- net /LCD_CS: track 0.00 -> 138.9 mm, vias 0 -> 3
- net /LCD_SDA: track 0.00 -> 138.1 mm, vias 0 -> 3
- net /LCD_DC: track 0.00 -> 131.9 mm, vias 0 -> 3
- net /LCD_RST: track 0.00 -> 131.1 mm, vias 0 -> 3
- net /LCD_BLK: track 0.00 -> 120.8 mm, vias 0 -> 4
- net Net-(U2-Vref): track 0.00 -> 90.0 mm, vias 0 -> 2
- net -12V: track 0.00 -> 87.7 mm, vias 0 -> 1
- net +12V: track 0.00 -> 68.6 mm, vias 0 -> 1
- net /VOWEL_POT: track 0.00 -> 56.7 mm, vias 0 -> 1
- net /MIDI_RX: track 0.00 -> 54.7 mm, vias 0 -> 1
- net /DAC_CS: track 0.00 -> 54.5 mm, vias 0 -> 1
- net /GATE: track 0.00 -> 52.6 mm, vias 0 -> 1
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- added copper zone on F.Cu, net GND
Other:
- board text added: "-12V"
- board text added: "tantricyphons"
- board text added: "tantricyphons crankery - dave hamilton rev 1 2026"

Commit message: ordered rev 1
Routing:
- net GND: track 2.23 -> 4.77 mm
- net /VREF_3V0_BUF: track 48.9 -> 50.3 mm
- net /ADC_DIN: track 39.4 -> 40.6 mm
- net /ENCODER_SW: track 49.1 -> 50.2 mm
- net +12V: track 68.6 -> 67.5 mm
- net /ENCODER_A: track 40.9 -> 41.6 mm
- net /MIDI_RX: track 54.7 -> 54.0 mm
- net +3.3V: track 156.0 -> 155.4 mm
