File: hw/control/control.kicad_pcb (KiCad board)
At the start: 2 copper layers, 196.3 x 128.5 mm, 97 parts, among them J1 1V/Oct, J11 Control D, J12 Control Pwr, J13 DAC Out, J14 Control A, J2 CV1, J3 CV2, J4 CV3, J5 CV4, J6 Vowel, J7 Gate, J8 MIDI IN, J9 Audio Out, SW1 Enc, SW2 Back, U1 6N138, U2 LM393, U3 TL074, U4 TL074

Commit message: kinda finsihed main
Parts:
- moved C3 2.54 mm to (81.3, 69.9)
- moved J11 2.54 mm to (86.4, 41.9)
- moved J13 2.54 mm to (86.4, 34.6)
- moved J14 2.54 mm to (86.4, 57.2)
Routing:
- removed copper zone on B.Cu, net (none)
Other:
- board size 196.3 x 128.5 mm -> 91.3 x 100 mm
- board text removed: "1"
- board text removed: "1V/Oct"
- board text removed: "2"
- board text removed: "3"
- board text removed: "4"
- board text removed: "Gate"
- board text removed: "MIDI"
- board text removed: "Out"
- board text removed: "Vowel"
- board text removed: "tantricyphons"
- board text removed: "↩"

Commit message: ordered rev 1
Parts:
- added LOGO3: crankery, lama:crankery_small, F.Cu at (111.1, 95.1)
- C8: value 1µF(Film) -> 1µF
- J11: footprint Connector_PinHeader_2.54mm:PinHeader_2x04_P2.54mm_Vertical -> lama:PinHeader_2x04_P2.54mm_Vertical
- J12: footprint Connector_PinHeader_2.54mm:PinHeader_1x06_P2.54mm_Vertical -> lama:PinHeader_1x06_P2.54mm_Vertical
- J13: footprint Connector_PinHeader_2.54mm:PinHeader_1x02_P2.54mm_Vertical -> lama:PinHeader_1x02_P2.54mm_Vertical
- J14: footprint Connector_PinHeader_2.54mm:PinHeader_2x07_P2.54mm_Vertical -> lama:PinHeader_2x07_P2.54mm_Vertical
- moved C3 7.63 mm to (88.9, 69.9)
- moved R24 2.54 mm to (30.3, 121.9)
- moved R25 2.54 mm to (27.7, 121.9)
- moved R29 2.54 mm to (51.1, 121.9)
- moved R30 2.54 mm to (48.6, 121.9)
- moved R40 2.54 mm to (111.0, 121.9)
- moved R43 2.54 mm to (113.6, 121.9)
- moved R41 2.33 mm to (35.4, 101.6), turned to 180 degrees
Routing:
- net /VREF_3V0_BUF: track 0.00 -> 232.1 mm, vias 0 -> 2
- net +5V: track 0.00 -> 135.6 mm, vias 0 -> 3
- net +3.3V: track 0.00 -> 119.9 mm, vias 0 -> 1
- net /EX_POT_{0}: track 0.00 -> 90.5 mm, vias 0 -> 1
- net Net-(U3A-+): track 0.00 -> 89.9 mm, vias 0 -> 1
- net Net-(R22-Pad1): track 0.00 -> 85.1 mm, vias 0 -> 1
- net Net-(U4D-+): track 0.00 -> 80.9 mm, vias 0 -> 1
- net /ENCODER_A: track 0.00 -> 78.6 mm, vias 0 -> 1
- net Net-(U3B--): track 0.00 -> 76.2 mm, vias 0 -> 3
- net /BACK_SW: track 0.00 -> 75.1 mm, vias 0 -> 2
- net /VOWEL_POT: track 0.00 -> 73.4 mm, vias 0 -> 1
- net Net-(U4B--): track 0.00 -> 73.3 mm, vias 0 -> 1
- net /ENCODER_B: track 0.00 -> 71.9 mm, vias 0 -> 1
- net /EX_POT_{1}: track 0.00 -> 67.9 mm, vias 0 -> 1
- net Net-(U4A--): track 0.00 -> 66.7 mm, vias 0 -> 2
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- added copper zone on F.Cu, net GND
Other:
- board text added: "tantricyphons"
- board text added: "tantricyphons crankery - dave hamilton rev 1 2026"
