File: hw/control/control.kicad_sch (KiCad schematic)
At the start: 98 parts, among them J1 1V/Oct, J11 Control D, J12 Control Pwr, J13 DAC Out, J14 Control A, J2 CV1, J3 CV2, J4 CV3, J5 CV4, J6 Vowel, J7 Gate, J8 MIDI IN, J9 Audio Out, SW1 Enc, SW2 Back, U1 6N138, U2 LM393, U3 TL074, U4 TL074

Commit message: ordered rev 1
Parts:
- added LOGO3: crankery, lama:crankery_small, symbol lama:Logo
- C8: value 1µF(Film) -> 1µF
- J11: footprint Connector_PinHeader_2.54mm:PinHeader_2x04_P2.54mm_Vertical -> lama:PinHeader_2x04_P2.54mm_Vertical
- J12: footprint Connector_PinHeader_2.54mm:PinHeader_1x06_P2.54mm_Vertical -> lama:PinHeader_1x06_P2.54mm_Vertical
- J13: footprint Connector_PinHeader_2.54mm:PinHeader_1x02_P2.54mm_Vertical -> lama:PinHeader_1x02_P2.54mm_Vertical
- J14: footprint Connector_PinHeader_2.54mm:PinHeader_2x07_P2.54mm_Vertical -> lama:PinHeader_2x07_P2.54mm_Vertical
Changed lines of the file:
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@@
 			)
 		)
-		(property "Footprint" "Connector_PinHeader_2.54mm:PinHeader_2x04_P2.54mm_Vertical"
+		(property "Footprint" "lama:PinHeader_2x04_P2.54mm_Vertical"
 			(at 115.57 176.53 0)
 			(hide yes)
@@
 			)
 		)
-		(property "Footprint" "Connector_PinHeader_2.54mm:PinHeader_2x07_P2.54mm_Vertical"
+		(property "Footprint" "lama:PinHeader_2x07_P2.54mm_Vertical"
 			(at 69.85 181.61 0)
 			(hide yes)
@@
 	)
 	(symbol
+		(lib_id "lama:Logo")
+		(at 160.02 185.42 0)
+		(unit 1)
+		(body_style 1)
+		(exclude_from_sim no)
+		(in_bom no)
+		(on_board yes)
+		(in_pos_files yes)
+		(dnp no)
+		(fields_autoplaced yes)
+		(property "Reference" "LOGO3"
+			(at 162.56 184.1499 0)
+			(show_name no)
+			(do_not_autoplace no)
+			(effects
+				(font
+					(size 1.27 1.27)
+				)
+				(justify left)
+			)
+		)
+		(property "Value" "crankery"
+			(at 162.56 186.6899 0)
+			(show_name no)
+			(do_not_autoplace no)
+			(effects
+				(font
+					(size 1.27 1.27)
+				)
+				(justify left)
+			)
+		)
+		(property "Footprint" "lama:crankery_small"
+			(at 160.02 185.42 0)
+			(hide yes)
+			(show_name no)
+			(do_not_autoplace no)
+			(effects
+				(font
+					(size 1.27 1.27)
+				)
+			)
+		)
+		(property "Datasheet" ""
+			(at 160.02 185.42 0)
+			(hide yes)
+			(show_name no)
+			(do_not_autoplace no)
+			(effects
+				(font
+					(size 1.27 1.27)
+				)
+			)
+		)
+		(property "Description" "Logo"
+			(at 160.02 185.42 0)
+			(hide yes)
+			(show_name no)
+			(do_not_autoplace no)
+			(effects
+				(font
+					(size 1.27 1.27)
+				)
+			)
+		)
+		(instances
+			(project "control"
+				(path "/d1915262-9239-4820-b50c-061fffa7cba0"
+					(reference "LOGO3")
+					(unit 1)
+				)
+			)
+		)
+	)
+	(symbol
 		(lib_id "power:+5V")
 		(at 219.71 21.59 0)
@@
 			)
 		)
-		(property "Footprint" "Connector_PinHeader_2.54mm:PinHeader_1x02_P2.54mm_Vertical"
+		(property "Footprint" "lama:PinHeader_1x02_P2.54mm_Vertical"
 			(at 156.21 173.99 0)
 			(hide yes)
@@
 			)
 		)
-		(property "Value" "1µF(Film)"
+		(property "Value" "1µF"
 			(at 205.74 130.81 90)
 			(show_name no)
@@
 			)
 		)
-		(property "Footprint" "Connector_PinHeader_2.54mm:PinHeader_1x06_P2.54mm_Vertical"
+		(property "Footprint" "lama:PinHeader_1x06_P2.54mm_Vertical"
 			(at 24.13 180.34 0)
 			(hide yes)
